Commit message: Add omnidirectional_controller to the simulation and Fix inertia problem

File: robot_description/urdf/holonomic_wheel/wheel.xacro (robot description, xacro)
@@ -1,4 +1,5 @@
 <?xml version="1.0"?>
 <robot xmlns:xacro="http://www.ros.org/wiki/xacro" >
+	<xacro:include filename="$(find robot_description)/urdf/standard_inertia_util.xacro" />
 	<xacro:property name="roue_xyz" value="0 0 0" />
 	<xacro:property name="roue_rpy" value="1.570796326794896558 1.570796326794896558 0" />
@@ -20,12 +21,16 @@
 				</geometry>
 			</collision>
-			<inertial>
+			<xacro:inertial_cylinder mass="0.073" length="0.0215" radius="0.03">
 				<origin xyz="-2.5184848675754577033e-17 4.8001766176252168599e-18 -0.0090500000000000198341" rpy="0 0 0"/>
-				<mass value="0.056036470001344637626" />
-				<inertia ixx="0.0" ixy="0.0"  ixz="0.0" iyy="1.0e-05" iyz="0.0" izz="0.0" />
-			</inertial>
+			</xacro:inertial_cylinder>
 		</link>
 		<gazebo reference="${name_roueholonome}">
 			<material>Gazebo/Grey</material>
+			<mu1>100.0</mu1>
+    		<mu2>100.8</mu2>
+			<kp>500000.0</kp>
+    		<kd>10.0</kd>
+			<min_depth>0.1</min_depth>
+			<maxVel>0.1</maxVel>
 		</gazebo>
 		<link name="rouleau_1_${name_roueholonome}">
@@ -45,16 +50,16 @@
 				</geometry>
 			</collision>
-			<inertial>
-				<origin xyz="-1.3533020587659002873e-19 -6.9388939039072283776e-18 -7.6373245842409416038e-17" rpy="0 0 0"/>
-				<mass value="0.0023432187849480503455" />
-				<inertia ixx="0.0" ixy="0.0"  ixz="0.0" iyy="8.1e-08" iyz="0.0" izz="0.0" />
-			</inertial>
+			<xacro:inertial_cylinder mass="0.010" length="0.019" radius="0.0075">
+            	<origin xyz="-1.3533020587659002873e-19 -6.9388939039072283776e-18 -7.6373245842409416038e-17" rpy="0 0 0"/>
+        	</xacro:inertial_cylinder>
 		</link>
 		<gazebo reference="rouleau_1_${name_roueholonome}">
 			<material>Gazebo/Black</material>
-			<mu1>1.0</mu1>
-    		<mu2>0.8</mu2>
-			<kp>1000.0</kp>
-    		<kd>10000.0</kd>
+			<mu1>100.0</mu1>
+    		<mu2>100.8</mu2>
+			<kp>500000.0</kp>
+    		<kd>10.0</kd>
+			<min_depth>0.1</min_depth>
+			<maxVel>0.1</maxVel>
 		</gazebo>
 		<joint name="Rouleau_a_${name_roueholonome}" type="continuous">
@@ -64,5 +69,5 @@
 			<axis xyz="0 0 1"/>
 			<limit effort="1" velocity="20" />
-			<joint_properties friction="0.0"/>
+			<joint_properties friction="10000.0"/>
 		</joint>
 		<link name="rouleau_2_${name_roueholonome}">
@@ -82,16 +87,16 @@
 				</geometry>
 			</collision>
-			<inertial>
+			<xacro:inertial_cylinder mass="0.010" length="0.019" radius="0.0075">
 				<origin xyz="-1.3533020587657876204e-19 3.4694469519536203518e-18 -6.6181745421045662032e-17" rpy="0 0 0"/>
-				<mass value="0.0023432187849480503455" />
-				<inertia ixx="0.0" ixy="0.0"  ixz="0.0" iyy="8.1e-08" iyz="0.0" izz="0.0" />
-			</inertial>
+			</xacro:inertial_cylinder>
 		</link>
 		<gazebo reference="rouleau_2_${name_roueholonome}">
 			<material>Gazebo/Black</material>
-			<mu1>1.0</mu1>
-    		<mu2>0.8</mu2>
-			<kp>1000.0</kp>
-    		<kd>10000.0</kd>
+			<mu1>100.0</mu1>
+    		<mu2>100.8</mu2>
+			<kp>500000.0</kp>
+    		<kd>10.0</kd>
+			<min_depth>0.1</min_depth>
+			<maxVel>0.1</maxVel>
 		</gazebo>
 		<joint name="Rouleau_b_${name_roueholonome}" type="continuous">
@@ -101,5 +106,5 @@
 			<axis xyz="0 0 1"/>
 			<limit effort="1" velocity="20" />
-			<joint_properties friction="0.0"/>
+			<joint_properties friction="10000.0"/>
 		</joint>
 		<link name="rouleau_3_${name_roueholonome}">
@@ -119,16 +124,16 @@
 				</geometry>
 			</collision>
-			<inertial>
+			<xacro:inertial_cylinder mass="0.010" length="0.019" radius="0.0075">
 				<origin xyz="-2.7890905821505490852e-17 -5.2041704279304320684e-18 -5.9242851517138445981e-17" rpy="0 0 0"/>
-				<mass value="0.0023432187849480503455" />
-				<inertia ixx="0.0" ixy="0.0"  ixz="0.0" iyy="8.1e-08" iyz="0.0" izz="0.0" />
-			</inertial>
+			</xacro:inertial_cylinder>
 		</link>
 		<gazebo reference="rouleau_3_${name_roueholonome}">
 			<material>Gazebo/Black</material>
-			<mu1>1.0</mu1>
-    		<mu2>0.8</mu2>
-			<kp>1000.0</kp>
-    		<kd>10000.0</kd>
+			<mu1>100.0</mu1>
+    		<mu2>100.8</mu2>
+			<kp>500000.0</kp>
+    		<kd>10.0</kd>
+			<min_depth>0.1</min_depth>
+			<maxVel>0.1</maxVel>
 		</gazebo>
 		<joint name="Rouleau_c_${name_roueholonome}" type="continuous">
@@ -138,5 +143,5 @@
 			<axis xyz="0 0 1"/>
 			<limit effort="1" velocity="20" />
-			<joint_properties friction="0.0"/>
+			<joint_properties friction="10000.0"/>
 		</joint>
 		<link name="rouleau_4_${name_roueholonome}">
@@ -156,16 +161,16 @@
 				</geometry>
 			</collision>
-			<inertial>
+			<xacro:inertial_cylinder mass="0.010" length="0.019" radius="0.0075">
 				<origin xyz="-1.3533020587658461205e-19 -5.2041704279304251351e-18 -5.5773404565184819466e-17" rpy="0 0 0"/>
-				<mass value="0.0023432187849480503455" />
-				<inertia ixx="0.0" ixy="0.0"  ixz="0.0" iyy="8.1e-08" iyz="0.0" izz="0.0" />
-			</inertial>
+			</xacro:inertial_cylinder>
 		</link>
 		<gazebo reference="rouleau_4_${name_roueholonome}">
 			<material>Gazebo/Black</material>
-			<mu1>1.0</mu1>
-    		<mu2>0.8</mu2>
-			<kp>1000.0</kp>
-    		<kd>10000.0</kd>
+			<mu1>100.0</mu1>
+    		<mu2>100.8</mu2>
+			<kp>500000.0</kp>
+    		<kd>10.0</kd>
+			<min_depth>0.1</min_depth>
+			<maxVel>0.1</maxVel>
 		</gazebo>
 		<joint name="Rouleau_d_${name_roueholonome}" type="continuous">
@@ -175,5 +180,5 @@
 			<axis xyz="0 0 1"/>
 			<limit effort="1" velocity="20" />
-			<joint_properties friction="0.0"/>
+			<joint_properties friction="10000.0"/>
 		</joint>
 		<link name="rouleau_5_${name_roueholonome}">
@@ -193,16 +198,16 @@
 				</geometry>
 			</collision>
-			<inertial>
+			<xacro:inertial_cylinder mass="0.010" length="0.019" radius="0.0075">
 				<origin xyz="-2.7890905821505497015e-17 3.4694469519536134185e-18 -5.9242851517138445981e-17" rpy="0 0 0"/>
-				<mass value="0.0023432187849480503455" />
-				<inertia ixx="0.0" ixy="0.0"  ixz="0.0" iyy="8.1e-08" iyz="0.0" izz="0.0" />
-			</inertial>
+			</xacro:inertial_cylinder>
 		</link>
 		<gazebo reference="rouleau_5_${name_roueholonome}">
 			<material>Gazebo/Black</material>
-			<mu1>1.0</mu1>
-    		<mu2>0.8</mu2>
-			<kp>1000.0</kp>
-    		<kd>10000.0</kd>
+			<mu1>100.0</mu1>
+    		<mu2>100.8</mu2>
+			<kp>500000.0</kp>
+    		<kd>10.0</kd>
+			<min_depth>0.1</min_depth>
+			<maxVel>0.1</maxVel>
 		</gazebo>
 		<joint name="Rouleau_e_${name_roueholonome}" type="continuous">
@@ -212,5 +217,5 @@
 			<axis xyz="0 0 1"/>
 			<limit effort="1" velocity="20" />
-			<joint_properties friction="0.0"/>
+			<joint_properties friction="10000.0"/>
 		</joint>
 		<link name="rouleau_6_${name_roueholonome}">
@@ -230,16 +235,16 @@
 				</geometry>
 			</collision>
-			<inertial>
+			<xacro:inertial_cylinder mass="0.010" length="0.019" radius="0.0075">
 				<origin xyz="-1.3533020587657560833e-19 -4.0005310894682744636e-33 -5.7508128041161638886e-17" rpy="0 0 0"/>
-				<mass value="0.0023432187849480503455" />
-				<inertia ixx="0.0" ixy="0.0"  ixz="0.0" iyy="8.1e-08" iyz="0.0" izz="0.0" />
-			</inertial>
+			</xacro:inertial_cylinder>
 		</link>
 		<gazebo reference="rouleau_6_${name_roueholonome}">
 			<material>Gazebo/Black</material>
-			<mu1>1.0</mu1>
-    		<mu2>0.8</mu2>
-			<kp>1000.0</kp>
-    		<kd>10000.0</kd>
+			<mu1>100.0</mu1>
+    		<mu2>100.8</mu2>
+			<kp>500000.0</kp>
+    	<kd>10.0</kd>
+			<min_depth>0.1</min_depth>
+			<maxVel>0.1</maxVel>
 		</gazebo>
 		<joint name="Rouleau_f_${name_roueholonome}" type="continuous">
@@ -249,5 +254,5 @@
 			<axis xyz="0 0 1"/>
 			<limit effort="1" velocity="20" />
-			<joint_properties friction="0.0"/>
+			<joint_properties friction="10000.0"/>
 		</joint>
 		<link name="rouleau_7_${name_roueholonome}">
@@ -267,16 +272,16 @@
 				</geometry>
 			</collision>
-			<inertial>
+			<xacro:inertial_cylinder mass="0.010" length="0.019" radius="0.0075">
 				<origin xyz="-1.3533020587658461205e-19 -6.9388939039072329999e-18 -5.750812804116162656e-17" rpy="0 0 0"/>
-				<mass value="0.0023432187849480503455" />
-				<inertia ixx="0.0" ixy="0.0"  ixz="0.0" iyy="8.1e-08" iyz="0.0" izz="0.0" />
-			</inertial>
+			</xacro:inertial_cylinder>
 		</link>
 		<gazebo reference="rouleau_7_${name_roueholonome}">
 			<material>Gazebo/Black</material>
-			<mu1>1.0</mu1>
-    		<mu2>0.8</mu2>
-			<kp>1000.0</kp>
-    		<kd>10000.0</kd>
+			<mu1>100.0</mu1>
+    		<mu2>100.8</mu2>
+			<kp>500000.0</kp>
+    		<kd>10.0</kd>
+			<min_depth>0.1</min_depth>
+			<maxVel>0.1</maxVel>
 		</gazebo>
 		<joint name="Rouleau_g_${name_roueholonome}" type="continuous">
@@ -286,5 +291,5 @@
 			<axis xyz="0 0 1"/>
 			<limit effort="1" velocity="20" />
-			<joint_properties friction="0.0"/>
+			<joint_properties friction="10000.0"/>
 		</joint>
 		<link name="rouleau_8_${name_roueholonome}">
@@ -304,16 +309,16 @@
 				</geometry>
 			</collision>
-			<inertial>
+			<xacro:inertial_cylinder mass="0.010" length="0.019" radius="0.0075">
 				<origin xyz="-1.3533020587658068797e-19 -1.0408340855860842566e-17 -6.6181745421045674358e-17" rpy="0 0 0"/>
-				<mass value="0.0023432187849480503455" />
-				<inertia ixx="0.0" ixy="0.0"  ixz="0.0" iyy="8.1e-08" iyz="0.0" izz="0.0" />
-			</inertial>
+			</xacro:inertial_cylinder>
 		</link>
 		<gazebo reference="rouleau_8_${name_roueholonome}">
 			<material>Gazebo/Black</material>
-			<mu1>1.0</mu1>
-    		<mu2>0.8</mu2>
-			<kp>1000.0</kp>
-    		<kd>10000.0</kd>
+			<mu1>100.0</mu1>
+    		<mu2>100.8</mu2>
+			<kp>500000.0</kp>
+    		<kd>10.0</kd>
+			<min_depth>0.1</min_depth>
+			<maxVel>0.1</maxVel>
 		</gazebo>
 		<joint name="Rouleau_h_${name_roueholonome}" type="continuous">
@@ -323,5 +328,5 @@
 			<axis xyz="0 0 1"/>
 			<limit effort="1" velocity="20" />
-			<joint_properties friction="0.0"/>
+			<joint_properties friction="10000.0"/>
 		</joint>
 		<link name="rouleau_9_${name_roueholonome}">
@@ -341,16 +346,16 @@
 				</geometry>
 			</collision>
-			<inertial>
+			<xacro:inertial_cylinder mass="0.010" length="0.019" radius="0.0075">
 				<origin xyz="-1.353302058765900528e-19 -8.1870457482636967244e-35 -6.5205963465808720368e-17" rpy="0 0 0"/>
-				<mass value="0.0023432187849480503455" />
-				<inertia ixx="0.0" ixy="0.0"  ixz="0.0" iyy="8.1e-08" iyz="0.0" izz="0.0" />
-			</inertial>
+			</xacro:inertial_cylinder>
 		</link>
 		<gazebo reference="rouleau_9_${name_roueholonome}">
 			<material>Gazebo/Black</material>
-			<mu1>1.0</mu1>
-    		<mu2>0.8</mu2>
-			<kp>1000.0</kp>
-    		<kd>10000.0</kd>
+			<mu1>100.0</mu1>
+    		<mu2>100.8</mu2>
+			<kp>500000.0</kp>
+    		<kd>10.0</kd>
+			<min_depth>0.1</min_depth>
+			<maxVel>0.1</maxVel>
 		</gazebo>
 		<joint name="Rouleau_i_${name_roueholonome}" type="continuous">
@@ -360,5 +365,5 @@
 			<axis xyz="0 0 1"/>
 			<limit effort="1" velocity="20" />
-			<joint_properties friction="0.0"/>
+			<joint_properties friction="10000.0"/>
 		</joint>
 		<link name="rouleau_10_${name_roueholonome}">
@@ -378,16 +383,16 @@
 				</geometry>
 			</collision>
-			<inertial>
+			<xacro:inertial_cylinder mass="0.010" length="0.019" radius="0.0075">
 				<origin xyz="-1.3533020587657876204e-19 6.4315019349350432793e-33 -5.9242851517138433655e-17" rpy="0 0 0"/>
-				<mass value="0.0023432187849480503455" />
-				<inertia ixx="0.0" ixy="0.0"  ixz="0.0" iyy="8.1e-08" iyz="0.0" izz="0.0" />
-			</inertial>
+			</xacro:inertial_cylinder>
 		</link>
 		<gazebo reference="rouleau_10_${name_roueholonome}">
 			<material>Gazebo/Black</material>
-			<mu1>1.0</mu1>
-    		<mu2>0.8</mu2>
-			<kp>1000.0</kp>
-    		<kd>10000.0</kd>
+			<mu1>100.0</mu1>
+    		<mu2>100.8</mu2>
+			<kp>500000.0</kp>
+    		<kd>10.0</kd>
+			<min_depth>0.1</min_depth>
+			<maxVel>0.1</maxVel>
 		</gazebo>
 		<joint name="Rouleau_j_${name_roueholonome}" type="continuous">
@@ -397,5 +402,5 @@
 			<axis xyz="0 0 1"/>
 			<limit effort="1" velocity="20" />
-			<joint_properties friction="0.0"/>
+			<joint_properties friction="10000.0"/>
 		</joint>
 		<joint name="joint_wheel_${name_roueholonome}" type="continuous">
@@ -405,5 +410,5 @@
 			<axis xyz="0 0 1"/>
 			<limit effort="1" velocity="20" />
-			<joint_properties friction="0.0"/>
+			<joint_properties friction="10000.0"/>
 		</joint>
 		<!-- <gazebo>

File: robot_description/urdf/robot.urdf (robot description, URDF)
Before this commit: robot robot, 35 links, 34 joints
Links:
- link roueholonome1: mass 0.056036470001344637626 -> 0.073
- link roueholonome2: mass 0.056036470001344637626 -> 0.073
- link roueholonome3: mass 0.056036470001344637626 -> 0.073
- link rouleau_10_roueholonome1: mass 0.0023432187849480503455 -> 0.01
- link rouleau_10_roueholonome2: mass 0.0023432187849480503455 -> 0.01
- link rouleau_10_roueholonome3: mass 0.0023432187849480503455 -> 0.01
- link rouleau_1_roueholonome1: mass 0.0023432187849480503455 -> 0.01
- link rouleau_1_roueholonome2: mass 0.0023432187849480503455 -> 0.01
- link rouleau_1_roueholonome3: mass 0.0023432187849480503455 -> 0.01
- link rouleau_2_roueholonome1: mass 0.0023432187849480503455 -> 0.01
- link rouleau_2_roueholonome2: mass 0.0023432187849480503455 -> 0.01
- link rouleau_2_roueholonome3: mass 0.0023432187849480503455 -> 0.01
- link rouleau_3_roueholonome1: mass 0.0023432187849480503455 -> 0.01
- link rouleau_3_roueholonome2: mass 0.0023432187849480503455 -> 0.01
- link rouleau_3_roueholonome3: mass 0.0023432187849480503455 -> 0.01
- link rouleau_4_roueholonome1: mass 0.0023432187849480503455 -> 0.01
- link rouleau_4_roueholonome2: mass 0.0023432187849480503455 -> 0.01
- link rouleau_4_roueholonome3: mass 0.0023432187849480503455 -> 0.01
- link rouleau_5_roueholonome1: mass 0.0023432187849480503455 -> 0.01
- link rouleau_5_roueholonome2: mass 0.0023432187849480503455 -> 0.01
- link rouleau_5_roueholonome3: mass 0.0023432187849480503455 -> 0.01
- link rouleau_6_roueholonome1: mass 0.0023432187849480503455 -> 0.01
- link rouleau_6_roueholonome2: mass 0.0023432187849480503455 -> 0.01
- link rouleau_6_roueholonome3: mass 0.0023432187849480503455 -> 0.01
- link rouleau_7_roueholonome1: mass 0.0023432187849480503455 -> 0.01
- link rouleau_7_roueholonome2: mass 0.0023432187849480503455 -> 0.01
- link rouleau_7_roueholonome3: mass 0.0023432187849480503455 -> 0.01
- link rouleau_8_roueholonome1: mass 0.0023432187849480503455 -> 0.01
- link rouleau_8_roueholonome2: mass 0.0023432187849480503455 -> 0.01
- link rouleau_8_roueholonome3: mass 0.0023432187849480503455 -> 0.01
- link rouleau_9_roueholonome1: mass 0.0023432187849480503455 -> 0.01
- link rouleau_9_roueholonome2: mass 0.0023432187849480503455 -> 0.01
- link rouleau_9_roueholonome3: mass 0.0023432187849480503455 -> 0.01

File: robot_description/urdf/robot.urdf.xacro (robot description, xacro)
@@ -2,6 +2,8 @@
 <robot xmlns:xacro="http://www.ros.org/wiki/xacro"  name="robot">
     <!-- Include all the contents. -->
-    <xacro:include filename="standard_inertia_util.xacro" />
-    <xacro:include filename="holonomic_wheel/wheel.xacro" />
+    <xacro:include filename="$(find robot_description)/urdf/standard_inertia_util.xacro" />
+    <xacro:include filename="$(find robot_description)/urdf/holonomic_wheel/wheel.xacro" />
+    <!-- <xacro:include filename="$(find robot_description)/urdf/gazebo.urdf.xacro"/> -->
+    <xacro:include filename="$(find robot_description)/urdf/ros2_control.urdf.xacro"/>
     <!-- This first link called "base_footprint" is empty -->
     <link name="base_footprint"/>
@@ -29,4 +31,11 @@
                 <mesh filename="file://$(find robot_description)/urdf/robot_base.stl"/>
             </geometry>
+            <surface>
+                <contact>
+                    <ode>
+                        <min_depth>0.001</min_depth>
+                    </ode>
+                </contact>
+            </surface>
         </collision>
 	    <xacro:inertial_cylinder mass="${mass}" length="${length}" radius="${radius}">
@@ -35,9 +44,11 @@
     </link>
     <gazebo reference="base_link">
-        <!--<material>Gazebo/Black</material>
+        <!-- <material>Gazebo/Black</material> -->
         <mu1>1.0</mu1>
-        <mu2>0.8</mu2> -->
-        <kp>1000.0</kp>
-        <kd>10000.0</kd>
+        <mu2>0.8</mu2>
+        <kp>500000.0</kp>
+        <kd>10.0</kd>
+        <min_depth>0.1</min_depth>
+        <maxVel>0.1</maxVel>
     </gazebo>
     <!-- Add the 3 holonomic wheel -->
@@ -48,3 +59,19 @@
     <xacro:holonomic_wheel joint_wheel_xyz="-0.11539788473061769747 0.06662500090107909001 0.018159998763917353098" joint_wheel_rpy="1.570796305932749215 3.6134297384305885703e-08 1.0471975360610779049" name_roueholonome="roueholonome3">
     </xacro:holonomic_wheel>
+    <gazebo>
+        <plugin filename="libgazebo_ros2_control.so" name="gazebo_ros2_control">
+            <robot_param>robot_description</robot_param>
+            <robot_param_node>robot_state_publisher</robot_param_node>
+            <parameters>$(find robot_nav)/params/omnidirectional_controller.yaml</parameters>
+        </plugin>
+        <plugin filename="libgazebo_ros_p3d.so" name="gazebo_ros_p3d" >
+            <ros>
+                <namespace>gazebo_ground_truth</namespace>
+            </ros>
+            <frame_name>world</frame_name>
+            <body_name>base_link</body_name>
+            <update_rate>50.0</update_rate>
+            <gaussian_noise>0.01</gaussian_noise>
+        </plugin>
+    </gazebo>
 </robot>
