Commit message: refactor: reorganises robot_description/urdf/ folder to move each stl and dae into his dedicated meshes/ folder

File: robot_description/urdf/holonomic_wheel/wheel.xacro (robot description, xacro)
@@ -9,5 +9,5 @@
 				<origin xyz= "${roue_xyz}" rpy="${roue_rpy}" />
 				<geometry>
-					<mesh filename="file://$(find robot_description)/urdf/holonomic_wheel/roueholonome.stl"/>
+					<mesh filename="file://$(find robot_description)/urdf/holonomic_wheel/meshes/roueholonome.stl"/>
 				</geometry>
 				<material name="roueholonome_material">
@@ -18,5 +18,5 @@
 				<origin xyz="${roue_xyz}" rpy="${roue_rpy}" />
 				<geometry>
-					<mesh filename="file://$(find robot_description)/urdf/holonomic_wheel/roueholonome.stl"/>
+					<mesh filename="file://$(find robot_description)/urdf/holonomic_wheel/meshes/roueholonome.stl"/>
 				</geometry>
 			</collision>
@@ -38,5 +38,5 @@
 				<origin xyz="0 -6.9388939039072283776e-18 -1.3660947373317355868e-17" rpy="-1.570796326794896558 7.4458241183643537248e-17 -2.2931001679521526839e-18" />
 				<geometry>
-					<mesh filename="file://$(find robot_description)/urdf/holonomic_wheel/rouleau.stl"/>
+					<mesh filename="file://$(find robot_description)/urdf/holonomic_wheel/meshes/rouleau.stl"/>
 				</geometry>
 				<material name="rouleau_material">
@@ -47,5 +47,5 @@
 				<origin xyz="0 -6.9388939039072283776e-18 -1.3660947373317355868e-17" rpy="-1.570796326794896558 7.4458241183643537248e-17 -2.2931001679521526839e-18" />
 				<geometry>
-					<mesh filename="file://$(find robot_description)/urdf/holonomic_wheel/rouleau.stl"/>
+					<mesh filename="file://$(find robot_description)/urdf/holonomic_wheel/meshes/rouleau.stl"/>
 				</geometry>
 			</collision>
@@ -75,5 +75,5 @@
 				<origin xyz="0 3.4694469519536141888e-18 -3.4694469519536141888e-18" rpy="-1.570796326794896558 1.704115477206629922e-17 1.0069492273628905161e-16" />
 				<geometry>
-					<mesh filename="file://$(find robot_description)/urdf/holonomic_wheel/rouleau.stl"/>
+					<mesh filename="file://$(find robot_description)/urdf/holonomic_wheel/meshes/rouleau.stl"/>
 				</geometry>
 				<material name="rouleau_material">
@@ -84,5 +84,5 @@
 				<origin xyz="0 3.4694469519536141888e-18 -3.4694469519536141888e-18" rpy="-1.570796326794896558 1.704115477206629922e-17 1.0069492273628905161e-16" />
 				<geometry>
-					<mesh filename="file://$(find robot_description)/urdf/holonomic_wheel/rouleau.stl"/>
+					<mesh filename="file://$(find robot_description)/urdf/holonomic_wheel/meshes/rouleau.stl"/>
 				</geometry>
 			</collision>
@@ -112,5 +112,5 @@
 				<origin xyz="-2.7755575615628913511e-17 -5.2041704279304212832e-18 3.4694469519536141888e-18" rpy="-1.57079632679489678 -3.8858620800219972321e-17 1.4515871623615415173e-17" />
 				<geometry>
-					<mesh filename="file://$(find robot_description)/urdf/holonomic_wheel/rouleau.stl"/>
+					<mesh filename="file://$(find robot_description)/urdf/holonomic_wheel/meshes/rouleau.stl"/>
 				</geometry>
 				<material name="rouleau_material">
@@ -121,5 +121,5 @@
 				<origin xyz="-2.7755575615628913511e-17 -5.2041704279304212832e-18 3.4694469519536141888e-18" rpy="-1.57079632679489678 -3.8858620800219972321e-17 1.4515871623615415173e-17" />
 				<geometry>
-					<mesh filename="file://$(find robot_description)/urdf/holonomic_wheel/rouleau.stl"/>
+					<mesh filename="file://$(find robot_description)/urdf/holonomic_wheel/meshes/rouleau.stl"/>
 				</geometry>
 			</collision>
@@ -149,5 +149,5 @@
 				<origin xyz="0 -5.2041704279304212832e-18 6.9388939039072283776e-18" rpy="-1.57079632679489678 2.2968870007964204446e-18 -1.2816475377239519703e-17" />
 				<geometry>
-					<mesh filename="file://$(find robot_description)/urdf/holonomic_wheel/rouleau.stl"/>
+					<mesh filename="file://$(find robot_description)/urdf/holonomic_wheel/meshes/rouleau.stl"/>
 				</geometry>
 				<material name="rouleau_material">
@@ -158,5 +158,5 @@
 				<origin xyz="0 -5.2041704279304212832e-18 6.9388939039072283776e-18" rpy="-1.57079632679489678 2.2968870007964204446e-18 -1.2816475377239519703e-17" />
 				<geometry>
-					<mesh filename="file://$(find robot_description)/urdf/holonomic_wheel/rouleau.stl"/>
+					<mesh filename="file://$(find robot_description)/urdf/holonomic_wheel/meshes/rouleau.stl"/>
 				</geometry>
 			</collision>
@@ -186,5 +186,5 @@
 				<origin xyz="-2.7755575615628913511e-17 3.4694469519536141888e-18 3.4694469519536141888e-18" rpy="-1.570796326794896558 -3.1610276974795425021e-18 9.1157131572497391962e-18" />
 				<geometry>
-					<mesh filename="file://$(find robot_description)/urdf/holonomic_wheel/rouleau.stl"/>
+					<mesh filename="file://$(find robot_description)/urdf/holonomic_wheel/meshes/rouleau.stl"/>
 				</geometry>
 				<material name="rouleau_material">
@@ -195,5 +195,5 @@
 				<origin xyz="-2.7755575615628913511e-17 3.4694469519536141888e-18 3.4694469519536141888e-18" rpy="-1.570796326794896558 -3.1610276974795425021e-18 9.1157131572497391962e-18" />
 				<geometry>
-					<mesh filename="file://$(find robot_description)/urdf/holonomic_wheel/rouleau.stl"/>
+					<mesh filename="file://$(find robot_description)/urdf/holonomic_wheel/meshes/rouleau.stl"/>
 				</geometry>
 			</collision>
@@ -223,5 +223,5 @@
 				<origin xyz="0 0 5.2041704279304212832e-18" rpy="-1.57079632679489678 -3.8858615837136297003e-17 1.4515871623615415173e-17" />
 				<geometry>
-					<mesh filename="file://$(find robot_description)/urdf/holonomic_wheel/rouleau.stl"/>
+					<mesh filename="file://$(find robot_description)/urdf/holonomic_wheel/meshes/rouleau.stl"/>
 				</geometry>
 				<material name="rouleau_material">
@@ -232,5 +232,5 @@
 				<origin xyz="0 0 5.2041704279304212832e-18" rpy="-1.57079632679489678 -3.8858615837136297003e-17 1.4515871623615415173e-17" />
 				<geometry>
-					<mesh filename="file://$(find robot_description)/urdf/holonomic_wheel/rouleau.stl"/>
+					<mesh filename="file://$(find robot_description)/urdf/holonomic_wheel/meshes/rouleau.stl"/>
 				</geometry>
 			</collision>
@@ -260,5 +260,5 @@
 				<origin xyz="0 -6.9388939039072283776e-18 5.2041704279304212832e-18" rpy="-1.57079632679489678 2.2968870007964204446e-18 -1.2816475377239519703e-17" />
 				<geometry>
-					<mesh filename="file://$(find robot_description)/urdf/holonomic_wheel/rouleau.stl"/>
+					<mesh filename="file://$(find robot_description)/urdf/holonomic_wheel/meshes/rouleau.stl"/>
 				</geometry>
 				<material name="rouleau_material">
@@ -269,5 +269,5 @@
 				<origin xyz="0 -6.9388939039072283776e-18 5.2041704279304212832e-18" rpy="-1.57079632679489678 2.2968870007964204446e-18 -1.2816475377239519703e-17" />
 				<geometry>
-					<mesh filename="file://$(find robot_description)/urdf/holonomic_wheel/rouleau.stl"/>
+					<mesh filename="file://$(find robot_description)/urdf/holonomic_wheel/meshes/rouleau.stl"/>
 				</geometry>
 			</collision>
@@ -297,5 +297,5 @@
 				<origin xyz="0 -1.0408340855860842566e-17 -3.4694469519536141888e-18" rpy="-1.570796326794896558 -3.1610276974795425021e-18 9.1157131572497391962e-18" />
 				<geometry>
-					<mesh filename="file://$(find robot_description)/urdf/holonomic_wheel/rouleau.stl"/>
+					<mesh filename="file://$(find robot_description)/urdf/holonomic_wheel/meshes/rouleau.stl"/>
 				</geometry>
 				<material name="rouleau_material">
@@ -306,5 +306,5 @@
 				<origin xyz="0 -1.0408340855860842566e-17 -3.4694469519536141888e-18" rpy="-1.570796326794896558 -3.1610276974795425021e-18 9.1157131572497391962e-18" />
 				<geometry>
-					<mesh filename="file://$(find robot_description)/urdf/holonomic_wheel/rouleau.stl"/>
+					<mesh filename="file://$(find robot_description)/urdf/holonomic_wheel/meshes/rouleau.stl"/>
 				</geometry>
 			</collision>
@@ -334,5 +334,5 @@
 				<origin xyz="0 0 -2.4936649967166601982e-18" rpy="-1.570796326794896558 7.4458252970967266128e-17 -2.2931034766746028961e-18" />
 				<geometry>
-					<mesh filename="file://$(find robot_description)/urdf/holonomic_wheel/rouleau.stl"/>
+					<mesh filename="file://$(find robot_description)/urdf/holonomic_wheel/meshes/rouleau.stl"/>
 				</geometry>
 				<material name="rouleau_material">
@@ -343,5 +343,5 @@
 				<origin xyz="0 0 -2.4936649967166601982e-18" rpy="-1.570796326794896558 7.4458252970967266128e-17 -2.2931034766746028961e-18" />
 				<geometry>
-					<mesh filename="file://$(find robot_description)/urdf/holonomic_wheel/rouleau.stl"/>
+					<mesh filename="file://$(find robot_description)/urdf/holonomic_wheel/meshes/rouleau.stl"/>
 				</geometry>
 			</collision>
@@ -371,5 +371,5 @@
 				<origin xyz="0 0 3.4694469519536141888e-18" rpy="-1.570796326794896558 1.704115477206629922e-17 1.0069492273628905161e-16" />
 				<geometry>
-					<mesh filename="file://$(find robot_description)/urdf/holonomic_wheel/rouleau.stl"/>
+					<mesh filename="file://$(find robot_description)/urdf/holonomic_wheel/meshes/rouleau.stl"/>
 				</geometry>
 				<material name="rouleau_material">
@@ -380,5 +380,5 @@
 				<origin xyz="0 0 3.4694469519536141888e-18" rpy="-1.570796326794896558 1.704115477206629922e-17 1.0069492273628905161e-16" />
 				<geometry>
-					<mesh filename="file://$(find robot_description)/urdf/holonomic_wheel/rouleau.stl"/>
+					<mesh filename="file://$(find robot_description)/urdf/holonomic_wheel/meshes/rouleau.stl"/>
 				</geometry>
 			</collision>

File: robot_description/urdf/lidar/lidar.xacro (robot description, xacro)
@@ -10,5 +10,5 @@
             <origin xyz="0.14618951398576332523 0.14013748441688259061 -0.032534567993216335913" rpy="0.0070131046609522990076 -0.0043951746943098691026 1.0588559938320413748e-20" />
             <geometry>
-                <mesh filename="file://$(find robot_description)/urdf/meshes/YDLidarX4.dae"/>
+                <mesh filename="file://$(find robot_description)/urdf/lidar/meshes/YDLidarX4.dae"/>
             </geometry>
             <cast_shadow>false</cast_shadow>
@@ -17,5 +17,5 @@
             <origin xyz="0.14618951398576332523 0.14013748441688259061 -0.032534567993216335913" rpy="0.0070131046609522990076 -0.0043951746943098691026 1.0588559938320413748e-20" />
             <geometry>
-                <mesh filename="file://$(find robot_description)/urdf/meshes/YDLidarX4.dae"/>
+                <mesh filename="file://$(find robot_description)/urdf/lidar/meshes/YDLidarX4.dae"/>
             </geometry>
         </collision>

File: robot_description/urdf/robot.urdf.xacro (robot description, xacro)
@@ -2,7 +2,7 @@
 <robot xmlns:xacro="http://www.ros.org/wiki/xacro"  name="robot">
     <!-- Include all the contents. -->
-    <xacro:include filename="$(find robot_description)/urdf/standard_inertia_util.xacro" />
+    <xacro:include filename="$(find robot_description)/urdf/meshes/standard_inertia_util.xacro" />
     <xacro:include filename="$(find robot_description)/urdf/holonomic_wheel/wheel.xacro" />
-    <xacro:include filename="$(find robot_description)/urdf/lidar.xacro" />
+    <xacro:include filename="$(find robot_description)/urdf/lidar/lidar.xacro" />
     <xacro:arg name="use_TopicBasedSystem_hardware_interface" default="false"/>
     <xacro:arg name="use_controller" default="false"/>
@@ -29,5 +29,5 @@
             <origin xyz="0 0 0" rpy="0 0 0"/>
             <geometry>
-                <mesh filename="file://$(find robot_description)/urdf/robot_base.stl"/>
+                <mesh filename="file://$(find robot_description)/urdf/meshes/robot_base.stl"/>
             </geometry>
             <material name="robot_base_material">
@@ -38,5 +38,5 @@
             <origin xyz="0 0 0" rpy="0 0 0" />
             <geometry>
-                <mesh filename="file://$(find robot_description)/urdf/robot_base.stl"/>
+                <mesh filename="file://$(find robot_description)/urdf/meshes/robot_base.stl"/>
             </geometry>
             <surface>
