Commit message: feat: Add laser_odometry launch file to bringup/

File: robot_description/urdf/lidar/lidar.xacro (robot description, xacro)
@@ -49,5 +49,5 @@
                     <type>gaussian</type>
                     <mean>0.0</mean>
-                    <stddev>0.004</stddev>
+                    <stddev>0.0005</stddev>
                 </noise>
             </ray>

File: robot_description/urdf/robot.urdf.xacro (robot description, xacro)
@@ -18,7 +18,7 @@
     <link name="base_footprint"/>
     <joint name="base_joint" type="fixed">
-        <origin xyz="0 0 -0.01" rpy="0 0 0"/>
-        <parent link="base_link"/>
-        <child link="base_footprint"/>
+        <origin xyz="0 0 0.01" rpy="0 0 0"/>
+        <parent link="base_footprint"/>
+        <child link="base_link"/>
     </joint>
     <xacro:property name="length" value="0.01" />
