Commit message: Fix: base_footprint frame to set x axis between two wheels

File: robot_description/urdf/robot.urdf.xacro (robot description, xacro)
@@ -19,5 +19,5 @@
     <link name="base_footprint"/>
     <joint name="base_joint" type="fixed">
-        <origin xyz="0 0 0.01" rpy="0 0 0"/>
+        <origin xyz="0 0 0.01" rpy="0 0 0.523599"/>
         <parent link="base_footprint"/>
         <child link="base_link"/>

Commit message: Fix: use of gpu with gazebo by adding __GLX_VENDOR_LIBRARY_NAME=nvidia and __NV_PRIME_RENDER_OFFLOAD=1 variables to bashrc, update base_link visual

File: robot_description/urdf/robot.urdf.xacro (robot description, xacro)
@@ -30,5 +30,5 @@
             <origin xyz="0 0 0" rpy="0 0 0"/>
             <geometry>
-                <mesh filename="file://$(find robot_description)/urdf/meshes/robot_base.stl"/>
+                <mesh filename="file://$(find robot_description)/urdf/meshes/robot_base.dae"/>
             </geometry>
             <material name="robot_base_material">
@@ -39,5 +39,5 @@
             <origin xyz="0 0 0" rpy="0 0 0" />
             <geometry>
-                <mesh filename="file://$(find robot_description)/urdf/meshes/robot_base.stl"/>
+                <mesh filename="file://$(find robot_description)/urdf/meshes/robot_base.dae"/>
             </geometry>
             <surface>
